Commit message: update the error of extract ORB pose, and PLICP params

File: turtlebot3/turtlebot3_description/urdf/turtlebot3_waffle.urdf.xacro (robot description, xacro)
@@ -140,5 +140,6 @@
     <parent link="base_link"/>
     <child link="base_scan"/>
-    <origin xyz="-0.064 0 0.122" rpy="0 0 0"/>
+    <!-- <origin xyz="-0.064 0 0.122" rpy="0 0 0"/> -->
+    <origin xyz="0.04 0 0.122" rpy="0 0 0"/>
   </joint>
   <link name="base_scan">
@@ -164,7 +165,12 @@
     </inertial>
   </link>
+  <!-- <joint name="camera_joint" type="fixed">
+    <origin xyz="0.064 -0.065 0.094" rpy="0 0 0"/>
+    <parent link="base_link"/>
+    <child link="camera_link"/>
+  </joint> -->
   <joint name="camera_joint" type="fixed">
-    <origin xyz="0.064 -0.065 0.094" rpy="0 0 0"/>
-    <parent link="base_link"/>
+    <origin xyz="0 0 0" rpy="0 0 0"/>
+    <parent link="base_scan"/>
     <child link="camera_link"/>
   </joint>

Commit message: change scan frame to base frame

File: turtlebot3/turtlebot3_description/urdf/turtlebot3_waffle.urdf.xacro (robot description, xacro)
@@ -142,7 +142,7 @@
     <child link="base_scan"/>
     <!-- sim -->
-    <!-- <origin xyz="0.0 0 0.122" rpy="0 0 0"/> -->
+    <origin xyz="0.0 0 0.122" rpy="0 0 0"/>
     <!-- original -->
-    <origin xyz="-0.064 0 0.122" rpy="0 0 0"/>
+    <!-- <origin xyz="-0.064 0 0.122" rpy="0 0 0"/> -->
   </joint>
   <link name="base_scan">
