Commit message: add simulation of bookstore and warehouse

File: turtlebot3/turtlebot3_description/urdf/turtlebot3_waffle.gazebo.xacro (robot description, xacro)
@@ -102,5 +102,5 @@
     </plugin>
   </gazebo>
-  <gazebo reference="base_scan">
+  <!-- <gazebo reference="base_scan">
     <material>Gazebo/FlatBlack</material>
     <sensor type="ray" name="lds_lfcd_sensor">
@@ -120,4 +120,36 @@
           <min>0.120</min>
           <max>3.5</max>
+          <resolution>0.015</resolution>
+        </range>
+        <noise>
+          <type>gaussian</type>
+          <mean>0.0</mean>
+          <stddev>0.01</stddev>
+        </noise>
+      </ray>
+      <plugin name="gazebo_ros_lds_lfcd_controller" filename="libgazebo_ros_laser.so">
+        <topicName>scan</topicName>
+        <frameName>base_scan</frameName>
+      </plugin>
+    </sensor>
+  </gazebo> -->
+  <gazebo reference="base_scan">
+    <material>Gazebo/FlatBlack</material>
+    <sensor type="ray" name="lds_lfcd_sensor">
+      <pose>0 0 0 0 0 0</pose>
+      <visualize>$(arg laser_visual)</visualize>
+      <update_rate>5</update_rate>
+      <ray>
+        <scan>
+          <horizontal>
+            <samples>360</samples>
+            <resolution>1</resolution>
+            <min_angle>0.0</min_angle>
+            <max_angle>6.28319</max_angle>
+          </horizontal>
+        </scan>
+        <range>
+          <min>0.120</min>
+          <max>10</max>
           <resolution>0.015</resolution>
         </range>

File: turtlebot3/turtlebot3_description/urdf/turtlebot3_waffle.urdf.xacro (robot description, xacro)
@@ -140,6 +140,6 @@
     <parent link="base_link"/>
     <child link="base_scan"/>
-    <!-- <origin xyz="-0.064 0 0.122" rpy="0 0 0"/> -->
-    <origin xyz="0.04 0 0.122" rpy="0 0 0"/>
+    <origin xyz="-0.064 0 0.122" rpy="0 0 0"/>
+    <!-- <origin xyz="0.04 0 0.122" rpy="0 0 0"/> -->
   </joint>
   <link name="base_scan">
@@ -171,5 +171,6 @@
   </joint> -->
   <joint name="camera_joint" type="fixed">
-    <origin xyz="0 0 0" rpy="0 0 0"/>
+    <!-- <origin xyz="-0.08 0.028 0.17" rpy="0 0 0"/> -->
+    <origin xyz="0 0 0.17" rpy="0 0 0"/>
     <parent link="base_scan"/>
     <child link="camera_link"/>

Commit message: add funtion untill compute precision, also do adjust ORB pose problem

File: turtlebot3/turtlebot3_description/urdf/turtlebot3_waffle.gazebo.xacro (robot description, xacro)
@@ -151,5 +151,5 @@
         <range>
           <min>0.120</min>
-          <max>10</max>
+          <max>3.5</max>
           <resolution>0.015</resolution>
         </range>
@@ -173,6 +173,10 @@
           <horizontal_fov>1.3439</horizontal_fov>
           <image>
-              <width>1920</width>
-              <height>1080</height>
+              <!-- <width>1920</width>
+              <height>1080</height> -->
+              <!-- <width>1280</width>
+              <height>720</height> -->
+              <width>640</width>
+              <height>480</height>
               <format>R8G8B8</format>
           </image>
@@ -186,5 +190,6 @@
         <baseline>0.2</baseline>
         <alwaysOn>true</alwaysOn>
-        <updateRate>30.0</updateRate>
+        <!-- <updateRate>30.0</updateRate> -->
+        <updateRate>200.0</updateRate>
         <cameraName>camera</cameraName>
         <frameName>camera_rgb_optical_frame</frameName>

File: turtlebot3/turtlebot3_description/urdf/turtlebot3_waffle.urdf.xacro (robot description, xacro)
@@ -137,12 +137,18 @@
   </joint>
   <link name="imu_link"/>
+  <!-- adjust this have some scan problem -->
   <joint name="scan_joint" type="fixed">
     <parent link="base_link"/>
     <child link="base_scan"/>
+    <!-- sim -->
+    <!-- <origin xyz="0.0 0 0.122" rpy="0 0 0"/> -->
+    <!-- original -->
     <origin xyz="-0.064 0 0.122" rpy="0 0 0"/>
-    <!-- <origin xyz="0.04 0 0.122" rpy="0 0 0"/> -->
   </joint>
   <link name="base_scan">
     <visual>
+      <!-- real world -->
+      <!-- <origin xyz="0.08 0 0" rpy="0 0 0"/> -->
+      <!-- sim -->
       <origin xyz="0 0 0" rpy="0 0 0"/>
       <geometry>
@@ -165,15 +171,25 @@
     </inertial>
   </link>
-  <!-- <joint name="camera_joint" type="fixed">
-    <origin xyz="0.064 -0.065 0.094" rpy="0 0 0"/>
-    <parent link="base_link"/>
+  <joint name="camera_joint" type="fixed">
+    <!-- real world -->
+    <!-- <origin xyz="0.064 -0.065 0.264" rpy="0 0 0"/> -->
+    <!-- sim -->
+      <!-- same with base_link -->
+    <!-- <origin xyz="0.0 0.0 0.264" rpy="0 0 0"/>' -->
+      <!-- same with scan link -->
+    <origin xyz="-0.064 0.0 0.264" rpy="0 0 0"/>'
+    <!-- <origin xyz="0.064 -0.065 0.264" rpy="0 0 0"/>' -->
+    <!-- original -->
+    <!-- <origin xyz="0.064 -0.065 0.094" rpy="0 0 0"/> -->
+    <parent link="base_link"/>
+    <child link="camera_link"/>
+  </joint>
+  <!-- adjust this xyz can change camera pose -->
+  <!-- <joint name="camera_joint" type="fixed"> -->
+    <!-- <origin xyz="-0.08 0.028 0.17" rpy="0 0 0"/> -->
+    <!-- <origin xyz="0 0 0.17" rpy="0 0 0"/>
+    <parent link="base_scan"/>
     <child link="camera_link"/>
   </joint> -->
-  <joint name="camera_joint" type="fixed">
-    <!-- <origin xyz="-0.08 0.028 0.17" rpy="0 0 0"/> -->
-    <origin xyz="0 0 0.17" rpy="0 0 0"/>
-    <parent link="base_scan"/>
-    <child link="camera_link"/>
-  </joint>
   <link name="camera_link">
     <visual>

Commit message: last update

File: turtlebot3/turtlebot3_description/urdf/turtlebot3_waffle.gazebo.xacro (robot description, xacro)
@@ -134,4 +134,36 @@
     </sensor>
   </gazebo> -->
+  <gazebo reference="base_scan2">
+    <material>Gazebo/FlatBlack</material>
+    <sensor type="ray" name="lds_lfcd_sensor">
+      <pose>0 0 0 0 0 0</pose>
+      <visualize>$(arg laser_visual)</visualize>
+      <update_rate>5</update_rate>
+      <ray>
+        <scan>
+          <horizontal>
+            <samples>360</samples>
+            <resolution>1</resolution>
+            <min_angle>0.0</min_angle>
+            <max_angle>6.28319</max_angle>
+          </horizontal>
+        </scan>
+        <range>
+          <min>0.120</min>
+          <max>8.0</max>
+          <resolution>0.015</resolution>
+        </range>
+        <noise>
+          <type>gaussian</type>
+          <mean>0.0</mean>
+          <stddev>0.01</stddev>
+        </noise>
+      </ray>
+      <plugin name="gazebo_ros_lds_lfcd_controller" filename="libgazebo_ros_laser.so">
+        <topicName>scan2</topicName>
+        <frameName>base_scan2</frameName>
+      </plugin>
+    </sensor>
+  </gazebo>
   <gazebo reference="base_scan">
     <material>Gazebo/FlatBlack</material>

File: turtlebot3/turtlebot3_description/urdf/turtlebot3_waffle.urdf.xacro (robot description, xacro)
@@ -238,3 +238,36 @@
   </joint>
   <link name="camera_depth_optical_frame"/>
+  <joint name="scan_joint2" type="fixed">
+    <parent link="base_link"/>
+    <child link="base_scan2"/>
+    <!-- sim -->
+    <origin xyz="0.0 0 0.122" rpy="0 0 0"/>
+    <!-- original -->
+    <!-- <origin xyz="-0.064 0 0.122" rpy="0 0 0"/> -->
+  </joint>
+  <link name="base_scan2">
+    <visual>
+      <!-- real world -->
+      <!-- <origin xyz="0.08 0 0" rpy="0 0 0"/> -->
+      <!-- sim -->
+      <origin xyz="0 0 0" rpy="0 0 0"/>
+      <geometry>
+        <mesh filename="package://turtlebot3_description/meshes/sensors/lds.stl" scale="0.001 0.001 0.001"/>
+      </geometry>
+      <material name="dark"/>
+    </visual>
+    <collision>
+      <origin xyz="0.015 0 -0.0065" rpy="0 0 0"/>
+      <geometry>
+        <cylinder length="0.0315" radius="0.055"/>
+      </geometry>
+    </collision>
+    <inertial>
+      <mass value="0.114" />
+      <origin xyz="0 0 0" />
+      <inertia ixx="0.001" ixy="0.0" ixz="0.0"
+               iyy="0.001" iyz="0.0"
+               izz="0.001" />
+    </inertial>
+  </link>
 </robot>
